Commit message: created waypoint navigation with Nav2

File: urdf/create3.urdf.xacro (robot description, xacro)
@@ -50,4 +50,13 @@
   <xacro:arg name="visualize_rays" default="false"/>
   <!-- Create 3 base definition-->
+   <!-- BASE_FOOTPRINT LINK -->
+    <joint name="base_footprint_joint" type="fixed">
+        <parent link="base_link"/>
+        <child link="base_footprint"/>
+        <origin xyz="0 0 0" rpy="0 0 0"/>
+    </joint>
+    <link name="base_footprint">
+    </link>
+    <!-- -->
   <link name="base_link">
     <visual>
